File: KiCAD Files for E-Skateboard/Electric Skateboard.kicad_pcb (KiCad board)
At the start: 2 copper layers, 130 x 140 mm, 25 parts, among them J1 ESP32 R, J10 SD Logger, J11 GPS, J12 UBEC, J2 ESP32 L, J3 Arduino Nano R, J4 Arduino Nano L, J5 Step Down, J6 ThumbTrigger, J7 ESC_Out, J8 Gyro, J9 OLED, Q1 IRLZ44N

Commit message: Ran DRC on PCB
Routing:
- net /3V3: track 562.0 -> 571.6 mm
- net /GPIO21: track 120.6 -> 118.1 mm
Changed lines of the file:
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@@
+	)
+	(segment
+		(start 136.08524 84.19748)
+		(end 136.19372 84.19748)
+		(width 0.2)
+		(layer "F.Cu")
+		(net 1)
 	)
 	(segment
@@
 	)
 	(segment
+		(start 141.401 89.40476)
+		(end 141.401 89.51324)
+		(width 0.2)
+		(layer "F.Cu")
+		(net 1)
+	)
+	(segment
 		(start 146.151 76.469)
 		(end 145 77.62)
@@
 	)
 	(segment
+		(start 136.19372 84.19748)
+		(end 141.401 89.40476)
+		(width 0.2)
+		(layer "F.Cu")
+		(net 1)
+	)
+	(segment
 		(start 133.980783 66.751)
 		(end 135.739 66.751)
@@
 	)
 	(segment
-		(start 136.08524 84.089)
-		(end 115.76524 104.409)
-		(width 0.2)
-		(layer "F.Cu")
-		(net 1)
-	)
-	(segment
 		(start 146.151 120.849)
 		(end 146.151 100.00324)
@@
 	)
 	(segment
-		(start 136.08524 84.19748)
-		(end 141.38776 89.5)
-		(width 0.2)
-		(layer "F.Cu")
-		(net 1)
-	)
-	(segment
 		(start 66 52.5)
 		(end 85.16 52.5)
@@
 	)
 	(segment
-		(start 115.76524 104.409)
-		(end 115.5 104.409)
-		(width 0.2)
-		(layer "F.Cu")
-		(net 1)
-	)
-	(segment
 		(start 57.295422 106.799)
 		(end 58.704578 106.799)
@@
 	)
 	(segment
+		(start 115.76524 104.409)
+		(end 136.08524 84.089)
+		(width 0.2)
+		(layer "F.Cu")
+		(net 1)
+	)
+	(segment
 		(start 135.739 71.79605)
 		(end 138.54395 74.601)
@@
 	)
 	(segment
+		(start 115.5 104.409)
+		(end 115.76524 104.409)
+		(width 0.2)
+		(layer "F.Cu")
+		(net 1)
+	)
+	(segment
 		(start 144.52324 99.329)
 		(end 141.38776 96.19352)
@@
 	)
 	(segment
+		(start 160.24 70)
+		(end 161.391 71.151)
+		(width 0.2)
+		(layer "F.Cu")
+		(net 2)
+	)
+	(segment
 		(start 146.552 125.448)
 		(end 146.552 116.708)
@@
 	)
 	(segment
-		(start 160.24 70)
-		(end 160.24 54.74)
-		(width 0.2)
-		(layer "F.Cu")
-		(net 2)
-	)
-	(segment
 		(start 86.92 108.48)
 		(end 86.92 127.5)
@@
 	)
 	(segment
+		(start 159.5 69.26)
+		(end 160.24 70)
+		(width 0.2)
+		(layer "F.Cu")
+		(net 2)
+	)
+	(segment
+		(start 161.391 76.469)
+		(end 160.24 77.62)
+		(width 0.2)
+		(layer "F.Cu")
+		(net 2)
+	)
+	(segment
 		(start 145 127)
 		(end 146.552 125.448)
@@
 	)
 	(segment
+		(start 159.5 54)
+		(end 159.5 69.26)
+		(width 0.2)
+		(layer "F.Cu")
+		(net 2)
+	)
+	(segment
 		(start 81.599 139.904)
 		(end 81.5 140.003)
@@
 	)
 	(segment
+		(start 161.391 71.151)
+		(end 161.391 76.469)
+		(width 0.2)
+		(layer "F.Cu")
+		(net 2)
+	)
+	(segment
 		(start 51.797 71.703)
 		(end 51.797 95)
@@
 	)
 	(segment
-		(start 94.54 127.5)
-		(end 93.02 129.02)
-		(width 0.2)
-		(layer "F.Cu")
-		(net 7)
-	)
-	(segment
 		(start 66 67.5)
 		(end 64.299 65.799)
@@
 		(width 0.2)
 		(layer "F.Cu")
-		(net 7)
-	)
-	(segment
-		(start 93.02 129.02)
-		(end 92.77 129.27)
-		(width 0.2)
-		(layer "F.Cu")
