File: PCB/Electric Skateboard.kicad_sch (KiCad schematic)
At the start: 21 parts, among them J1 ESP32 R, J10 SD Logger, J11 GPS, J12 UBEC, J2 ESP32 L, J3 Arduino Nano R, J4 Arduino Nano L, J5 Step Down, J6 ThumbTrigger, J7 ESC_Out, J8 Gyro, J9 OLED, Q1 IRLZ44N

Commit message: Changed File Organization, Added BOM
Parts:
- added R7: 100, Resistor_THT:R_Axial_DIN0207_L6.3mm_D2.5mm_P10.16mm_Horizontal, symbol Device:R
Connections:
- net 3V3: no longer BZ1.1 (+), J10.2 (Pin_2), J11.4 (Pin_4), J12.1 (Pin_1), J2.15 (Pin_15), J3.1 (Pin_1), J3.14 (Pin_14), J3.4 (Pin_4)
- net GPIO26: now also R7.2
- new net: BZ1.1 (+), R7.1
- new net 5V: J10.2 (Pin_2), J11.4 (Pin_4), J12.1 (Pin_1), J2.15 (Pin_15), J3.4 (Pin_4)
Other:
- moved on the sheet: BZ1, D1, J1, J10, J11, J12, J2, J3, J4, J5, J6, J7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
