File: PCB/Electric Skateboard.kicad_pcb (KiCad board)
At the start: 2 copper layers, 130 x 140 mm, 25 parts, among them J1 ESP32 R, J10 SD Logger, J11 GPS, J12 UBEC, J2 ESP32 L, J3 Arduino Nano R, J4 Arduino Nano L, J5 Step Down, J6 ThumbTrigger, J7 ESC_Out, J8 Gyro, J9 OLED, Q1 IRLZ44N

Commit message: Changed File Organization, Added BOM
Parts:
- added R7: 100, Resistor_THT:R_Axial_DIN0207_L6.3mm_D2.5mm_P10.16mm_Horizontal, F.Cu at (57.3, 80.5)
Connections:
- BZ1 pad 1: /3V3 -> Net-(BZ1-+)
- J10 pad 2: /3V3 -> /5V
- J11 pad 4: /3V3 -> /5V
- J12 pad 1: /3V3 -> /5V
- J2 pad 15: /3V3 -> /5V
- J3 pad 1: /3V3 -> unconnected-(J3-Pin_1-Pad1)
- J3 pad 14: /3V3 -> unconnected-(J3-Pin_14-Pad14)
- J3 pad 4: /3V3 -> /5V
Changed lines of the file:
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@@
 	(net 58 "unconnected-(J8-Pin_7-Pad7)")
 	(net 59 "/Gate")
+	(net 60 "Net-(BZ1-+)")
+	(net 61 "/5V")
+	(net 62 "unconnected-(J3-Pin_14-Pad14)")
+	(net 63 "unconnected-(J3-Pin_1-Pad1)")
 	(footprint "Resistor_THT:R_Axial_DIN0207_L6.3mm_D2.5mm_P10.16mm_Horizontal"
 		(layer "F.Cu")
@@
 			(layers "*.Cu" "*.Mask")
 			(remove_unused_layers no)
-			(net 2 "/3V3")
+			(net 63 "unconnected-(J3-Pin_1-Pad1)")
 			(pinfunction "Pin_1")
 			(pintype "passive")
@@
 			(layers "*.Cu" "*.Mask")
 			(remove_unused_layers no)
-			(net 2 "/3V3")
+			(net 61 "/5V")
 			(pinfunction "Pin_4")
 			(pintype "passive")
@@
 			(layers "*.Cu" "*.Mask")
 			(remove_unused_layers no)
-			(net 2 "/3V3")
+			(net 62 "unconnected-(J3-Pin_14-Pad14)")
 			(pinfunction "Pin_14")
 			(pintype "passive")
@@
 			(remove_unused_layers no)
 			(roundrect_rratio 0.089286)
-			(net 2 "/3V3")
+			(net 61 "/5V")
 			(pinfunction "Pin_1")
 			(pintype "passive")
@@
 			(layers "*.Cu" "*.Mask")
 			(remove_unused_layers no)
-			(net 2 "/3V3")
+			(net 61 "/5V")
 			(pinfunction "Pin_4")
 			(pintype "passive")
@@
 			(layers "*.Cu" "*.Mask")
 			(remove_unused_layers no)
-			(net 2 "/3V3")
+			(net 61 "/5V")
 			(pinfunction "Pin_15")
 			(pintype "passive")
@@
 			(layers "*.Cu" "*.Mask")
 			(remove_unused_layers no)
-			(net 2 "/3V3")
+			(net 61 "/5V")
 			(pinfunction "Pin_2")
 			(pintype "passive")
@@
 	(footprint "Resistor_THT:R_Axial_DIN0207_L6.3mm_D2.5mm_P10.16mm_Horizontal"
 		(layer "F.Cu")
+		(at 57.34 80.5)
+		(descr "Resistor, Axial_DIN0207 series, Axial, Horizontal, pin pitch=10.16mm, 0.25W = 1/4W, length*diameter=6.3*2.5mm^2, http://cdn-reichelt.de/documents/datenblatt/B400/1_4W%23YAG.pdf")
+		(tags "Resistor Axial_DIN0207 series Axial Horizontal pin pitch 10.16mm 0.25W = 1/4W length 6.3mm diameter 2.5mm")
+		(property "Reference" "R7"
+			(at 5.08 -2.37 0)
+			(layer "F.SilkS")
+			(effects
+				(font
+					(size 1 1)
+					(thickness 0.15)
+				)
+			)
+		)
+		(property "Value" "100"
+			(at 5.08 2.37 0)
+			(layer "F.Fab")
+			(effects
+				(font
+					(size 1 1)
+					(thickness 0.15)
+				)
+			)
+		)
+		(property "Datasheet" "~"
+			(at 0 0 0)
+			(layer "F.Fab")
+			(hide yes)
+			(effects
+				(font
+					(size 1.27 1.27)
+					(thickness 0.15)
+				)
+			)
+		)
+		(property "Description" "Resistor"
+			(at 0 0 0)
+			(layer "F.Fab")
+			(hide yes)
+			(effects
+				(font
+					(size 1.27 1.27)
+					(thickness 0.15)
+				)
+			)
+		)
+		(property ki_fp_filters "R_*")
+		(sheetname "/")
+		(sheetfile "Electric Skateboard.kicad_sch")
+		(attr through_hole)
+		(fp_line
+			(start 1.04 0)
+			(end 1.81 0)
+			(stroke
+				(width 0.12)
+				(type solid)
+			)
+			(layer "F.SilkS")
+		)
+		(fp_line
+			(start 9.12 0)
+			(end 8.35 0)
+			(stroke
+				(width 0.12)
+				(type solid)
+			)
+			(layer "F.SilkS")
+		)
+		(fp_rect
+			(start 1.81 -1.37)
+			(end 8.35 1.37)
+			(stroke
+				(width 0.12)
+				(type solid)
+			)
+			(fill no)
+			(layer "F.SilkS")
+		)
+		(fp_rect
+			(start -1.05 -1.5)
+			(end 11.21 1.5)
+			(stroke
+				(width 0.05)
+				(type solid)
+			)
+			(fill no)
+			(layer "F.CrtYd")
+		)
+		(fp_line
+			(start 0 0)
+			(end 1.93 0)
+			(stroke
+				(width 0.1)
+				(type solid)
+			)
+			(layer "F.Fab")
+		)
+		(fp_line
+			(start 10.16 0)
+			(end 8.23 0)
+			(stroke
+				(width 0.1)
+				(type solid)
+			)
+			(layer "F.Fab")
+		)
+		(fp_rect
+			(start 1.93 -1.25)
+			(end 8.23 1.25)
+			(stroke
+				(width 0.1)
+				(type solid)
+			)
+			(fill no)
+			(layer "F.Fab")
+		)
+		(fp_text user "${REFERENCE}"
+			(at 5.08 0 0)
+			(layer "F.Fab")
+			(effects
+				(font
+					(size 1 1)
+					(thickness 0.15)
+				)
+			)
+		)
+		(pad "1" thru_hole circle
+			(at 0 0)
+			(size 1.6 1.6)
+			(drill 0.8)
+			(layers "*.Cu" "*.Mask")
+			(remove_unused_layers no)
+			(net 60 "Net-(BZ1-+)")
+			(pintype "passive")
+		)
+		(pad "2" thru_hole circle
+			(at 10.16 0)
+			(size 1.6 1.6)
+			(drill 0.8)
+			(layers "*.Cu" "*.Mask")
+			(remove_unused_layers no)
+			(net 24 "/GPIO26")
+			(pintype "passive")
+		)
+		(embedded_fonts no)
+		(model "${KICAD9_3DMODEL_DIR}/Resistor_THT.3dshapes/R_Axial_DIN0207_L6.3mm_D2.5mm_P10.16mm_Horizontal.step"
+			(offset
+				(xyz 0 0 0)
+			)
+			(scale
+				(xyz 1 1 1)
+			)
+			(rotate
+				(xyz 0 0 0)
+			)
+		)
+	)
+	(footprint "Resistor_THT:R_Axial_DIN0207_L6.3mm_D2.5mm_P10.16mm_Horizontal"
+		(layer "F.Cu")
 		(at 96 73.5 90)
 		(descr "Resistor, Axial_DIN0207 series, Axial, Horizontal, pin pitch=10.16mm, 0.25W = 1/4W, length*diameter=6.3*2.5mm^2, http://cdn-reichelt.de/documents/datenblatt/B400/1_4W%23YAG.pdf")
@@
 			(layers "*.Cu" "*.Mask")
 			(remove_unused_layers no)
-			(net 2 "/3V3")
+			(net 60 "Net-(BZ1-+)")
 			(pinfunction "+")
 			(pintype "passive")

Commit message: Fixed PCB
Parts:
- removed the REF** at (53.9, 32.6)
- removed the REF** at (167.9, 32.6)
- removed the REF** at (53.9, 156.6)
- removed the REF** at (167.9, 156.6)
- added REF**: MountingHole_5.3mm_M5, MountingHole:MountingHole_5.3mm_M5, F.Cu at (166.9, 157.6)
- added REF**: MountingHole_5.3mm_M5, MountingHole:MountingHole_5.3mm_M5, F.Cu at (52.9, 157.6)
- added REF**: MountingHole_5.3mm_M5, MountingHole:MountingHole_5.3mm_M5, F.Cu at (52.9, 33.6)
- added REF**: MountingHole_5.3mm_M5, MountingHole:MountingHole_5.3mm_M5, F.Cu at (166.9, 33.6)
- moved BZ1 1.41 mm to (54.7, 96.0)
- moved D1 1.41 mm to (133.0, 38.5)
- moved J1 1.41 mm to (105.9, 71.0)
- moved J10 1.41 mm to (139.0, 128.0)
- moved J11 1.41 mm to (143.5, 55.0)
- moved J12 1.41 mm to (92.8, 55.0)
- moved J2 1.41 mm to (83.0, 71.0)
- moved J3 1.41 mm to (159.2, 71.0)
- moved J4 1.41 mm to (144.0, 71.0)
- moved J5 1.41 mm to (119.0, 55.0)
- moved J6 1.41 mm to (57.0, 119.5)
- moved J7 1.41 mm to (57.0, 138.5)
- moved J8 1.41 mm to (85.9, 128.5)
- moved J9 1.41 mm to (65.0, 68.5)
- moved Q1 1.41 mm to (131.0, 66.5)
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Routing:
- net /3V3: track 571.6 -> 110.8 mm
- net /5V: track 0.00 -> 202.1 mm
- net /GPIO26: track 0.00 -> 75.2 mm
- net Net-(BZ1-+): track 0.00 -> 15.1 mm
